File: PCB/Model C-1.0.kicad_pcb (KiCad board)
At the start: 2 copper layers, 80 x 145 mm, 49 parts, among them J1 1.5V-5V Boost Converter, J3 AVR-ISP-6, J4 reset, J5 boot, SW1 SW_SPST, U1 ATmega32A-A, U3 CA56-12CGKWA, U4 CA56-12CGKWA, U5 MAX7219, Y1 Crystal

Commit message: better pcb with the right components - maybe final?
Parts:
- BT1: footprint Battery:BatteryHolder_Keystone_1058_1x2032 -> Battery:BatteryHolder_Keystone_2466_1xAAA
- SW1: footprint Button_Switch_SMD:SW_SPST_TL3305A -> Button_Switch_THT:SW_CuK_OS102011MA1QN1_SPDT_Angled
- U5: footprint Package_DIP:DIP-24_W7.62mm_SMDSocket_SmallPads -> Package_SO:SSOP-24_3.9x8.7mm_P0.635mm
- moved BT1 10.0 mm to (53.4, 61.1), turned to 0 degrees
- moved U5 7.65 mm to (91.6, 49.3)
- moved R11 4.88 mm to (91.4, 44.6)
- moved SW1 3.16 mm to (101.2, 79.1)
Routing:
- net Net-(BT1-+): track 23.5 -> 44.3 mm
- net /sck: track 91.2 -> 78.8 mm
- net /7: track 64.4 -> 75.7 mm
- net /6: track 38.7 -> 49.4 mm, vias 2 -> 0
- net /3: track 21.2 -> 31.0 mm
- net /2: track 12.0 -> 21.7 mm
- net /mosi: track 57.4 -> 66.3 mm
- net /ssg: track 81.7 -> 72.8 mm
- net /b: track 52.0 -> 60.4 mm, vias 0 -> 2
- net /a: track 74.7 -> 82.1 mm, vias 2 -> 3
- net /0: track 49.0 -> 42.6 mm
- net /5: track 55.8 -> 61.8 mm
- net /d: track 74.3 -> 79.3 mm, vias 1 -> 3
- net /c: track 77.9 -> 82.9 mm, vias 1 -> 0
- net /g: track 79.0 -> 83.4 mm
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
Commit message: mounting holes + clean drc
Parts:
- added H1: MountingHole, MountingHole:MountingHole_3.2mm_M3, F.Cu at (29.9, 42.5)
- added H2: MountingHole, MountingHole:MountingHole_3.2mm_M3, F.Cu at (104.7, 42.5)
- added H3: MountingHole, MountingHole:MountingHole_3.2mm_M3, F.Cu at (29.9, 182.4)
- added H4: MountingHole, MountingHole:MountingHole_3.2mm_M3, F.Cu at (29.8, 85.8)
- added H5: MountingHole, MountingHole:MountingHole_3.2mm_M3, F.Cu at (29.9, 92.9)
- added H6: MountingHole, MountingHole:MountingHole_3.2mm_M3, F.Cu at (104.7, 92.3)
- added H7: MountingHole, MountingHole:MountingHole_3.2mm_M3, F.Cu at (104.7, 85.5)
- added H8: MountingHole, MountingHole:MountingHole_3.2mm_M3, F.Cu at (104.8, 182.6)
- added H9: MountingHole, MountingHole:MountingHole_3.2mm_M3, F.Cu at (66.8, 126.2)
Routing:
- net GND: track 28.7 -> 50.5 mm, vias 33 -> 34
- net /row1: track 145.4 -> 149.6 mm
- net /col0: track 121.4 -> 124.9 mm
- net /col1: track 113.8 -> 110.4 mm
- net /col3: track 157.4 -> 154.0 mm
- net /col2: track 149.7 -> 146.3 mm
